File: FunkyHat/FunkyHat.sch (KiCad schematic (older format))
At the start: 47 parts, among them J1 Conn_Coaxial, J3 40HAT, J6 CONN_02X02, J9 CONN_01X02, Q1 DMG2305UX, Q2 DMMT5401, U2 CAT24C32

Commit message: Doku erweitert, Schaltplan fortgesetzt
Parts:
- added D1: LED_RGBA, symbol Device:LED_RGBA
- added R1, R2, R3: 220Ω, symbol Device:R
- U?: symbol ATMEGA128RFA1-ZU:ATMEGA128RFA1-ZU -> FunkyHat-rescue:ATMEGA128RFA1-ZU-ATMEGA128RFA1-ZU
- U?: symbol RC522:RC522 -> FunkyHat-rescue:RC522-RC522
Connections:
- net 3.3V_EEPROM: now also D1.4 (A)
- new net: D1.1 (RK), R1.1
- new net: D1.2 (GK), R2.1
- new net: D1.3 (BK), R3.1
Other:
- note added: "Anschluss an RPi oder Micro-Controller?"
- note added: "RGB-LED"
- moved on the sheet: U?
Changed lines of the file:
@@
 Bleibt drin, weil wer weiß was passiert\nwenn ich das lösche... (MS)
 $Comp
-L ATMEGA128RFA1-ZU:ATMEGA128RFA1-ZU U?
+L FunkyHat-rescue:ATMEGA128RFA1-ZU-ATMEGA128RFA1-ZU U?
 U 1 1 60165848
 P 7350 11300
@@
 Text Notes 4700 8400 0    79   ~ 16
 Microcontroller
-Text Notes 18500 1950 0    79   ~ 16
+Text Notes 10500 850  0    79   ~ 16
 NFC/RFID Chip
 $Comp
-L RC522:RC522 U?
+L FunkyHat-rescue:RC522-RC522 U?
 U 1 1 60194D96
-P 19750 3400
-F 0 "U?" H 19750 4767 50  0000 C CNN
-F 1 "RC522" H 19750 4676 50  0000 C CNN
-F 2 "QFN50P500X500X100-33N" H 19750 3400 50  0001 L BNN
-F 3 "" H 19750 3400 50  0001 L BNN
-F 4 "1mm" H 19750 3400 50  0001 L BNN "MAXIMUM_PACKAGE_HIEGHT"
-F 5 "IPC7351B" H 19750 3400 50  0001 L BNN "STANDARD"
-F 6 "NXP USA" H 19750 3400 50  0001 L BNN "MANUFACTURER"
-F 7 "3.9" H 19750 3400 50  0001 L BNN "PARTREV"
-	1    19750 3400
+P 12950 2600
+F 0 "U?" H 12950 3967 50  0000 C CNN
+F 1 "RC522" H 12950 3876 50  0000 C CNN
+F 2 "QFN50P500X500X100-33N" H 12950 2600 50  0001 L BNN
+F 3 "" H 12950 2600 50  0001 L BNN
+F 4 "1mm" H 12950 2600 50  0001 L BNN "MAXIMUM_PACKAGE_HIEGHT"
+F 5 "IPC7351B" H 12950 2600 50  0001 L BNN "STANDARD"
+F 6 "NXP USA" H 12950 2600 50  0001 L BNN "MANUFACTURER"
+F 7 "3.9" H 12950 2600 50  0001 L BNN "PARTREV"
+	1    12950 2600
 	1    0    0    -1
 $EndComp
@@
 Wire Notes Line
 	4700 950  10350 950
-Text GLabel 5300 8650 0    50   Input ~ 0
-GND_GPIO_7
 Text GLabel 5300 8750 0    50   Input ~ 0
 5V_HAT
@@
 Wire Notes Line
 	500  14350 500  10900
+Text Notes 10500 5700 0    79   ~ 16
+RGB-LED
+Text GLabel 11400 1350 0    50   Input ~ 0
+GND_GPIO_8
+Text GLabel 11400 1450 0    50   Input ~ 0
+3.3V_EEPROM
+Text GLabel 5300 8650 0    50   Input ~ 0
+GND_GPIO_7
+$Comp
+L Device:LED_RGBA D1
+U 1 1 6048F38A
+P 11800 6450
+F 0 "D1" H 11800 6947 50  0000 C CNN
+F 1 "LED_RGBA" H 11800 6856 50  0000 C CNN
+F 2 "" H 11800 6400 50  0001 C CNN
+F 3 "~" H 11800 6400 50  0001 C CNN
+	1    11800 6450
+	1    0    0    -1
+$EndComp
+Text GLabel 12150 6450 2    50   Input ~ 0
+3.3V_EEPROM
+$Comp
+L Device:R R1
+U 1 1 6051728B
+P 11450 6150
+F 0 "R1" V 11243 6150 50  0000 C CNN
+F 1 "220Ω" V 11334 6150 50  0000 C CNN
+F 2 "" V 11380 6150 50  0001 C CNN
+F 3 "~" H 11450 6150 50  0001 C CNN
+	1    11450 6150
+	0    1    1    0
+$EndComp
+$Comp
+L Device:R R2
+U 1 1 60519DE7
+P 11450 6450
+F 0 "R2" V 11243 6450 50  0000 C CNN
+F 1 "220Ω" V 11334 6450 50  0000 C CNN
+F 2 "" V 11380 6450 50  0001 C CNN
+F 3 "~" H 11450 6450 50  0001 C CNN
+	1    11450 6450
+	0    1    1    0
+$EndComp
+$Comp
+L Device:R R3
+U 1 1 60523EA3
+P 11450 6750
+F 0 "R3" V 11243 6750 50  0000 C CNN
+F 1 "220Ω" V 11334 6750 50  0000 C CNN
+F 2 "" V 11380 6750 50  0001 C CNN
+F 3 "~" H 11450 6750 50  0001 C CNN
+	1    11450 6750
+	0    1    1    0
+$EndComp
+Wire Wire Line
+	11600 6650 11600 6750
+Wire Wire Line
+	11600 6250 11600 6150
+Wire Wire Line
+	12150 6450 12000 6450
+Wire Wire Line
+	11300 6150 11150 6150
+Wire Wire Line
+	11300 6450 11150 6450
+Wire Wire Line
+	11300 6750 11150 6750
+Wire Notes Line
+	10500 950  10500 5500
+Wire Notes Line
+	10500 5500 16500 5500
+Wire Notes Line
+	16500 5500 16500 950
+Wire Notes Line
+	16500 950  10500 950
+Wire Notes Line
+	10500 5750 12750 5750
+Wire Notes Line
+	12750 5750 12750 7500
+Wire Notes Line
+	12750 7500 10500 7500
+Wire Notes Line
+	10500 7500 10500 5750
+Text Notes 10550 5850 0    50   ~ 0
+Anschluss an RPi oder Micro-Controller?
 $EndSCHEMATC
